File: Stylophon_1.kicad_pcb (KiCad board)
At the start: 2 copper layers, 57 x 38.5 mm, 70 parts, among them J4 Stylus, SW1 On/Off, SW2 Vibrato, T1 BC846, T2 BC846, U1 NE555D

Commit message: VIA stitching & GND Plane QR
Parts:
- added TP21: 9V, TestPoint:TestPoint_Pad_D1.5mm, B.Cu at (146.5, 88.4)
- added TP22: GND, TestPoint:TestPoint_Pad_D1.5mm, B.Cu at (139.0, 94.0)
- added TP23: Output, TestPoint:TestPoint_Pad_D1.5mm, B.Cu at (154.9, 88.1)
- added TP24: Sinus, TestPoint:TestPoint_Pad_D1.5mm, B.Cu at (129.0, 85.0)
- added TP25: Batterie, TestPoint:TestPoint_Pad_D1.5mm, B.Cu at (116.2, 94.1)
Routing:
- net GND: track 77.8 -> 96.4 mm, vias 2 -> 39
- net +9V: track 115.1 -> 120.6 mm, vias 0 -> 2
- net Net-(U1-Q): track 8.26 -> 11.3 mm, vias 0 -> 1
- net Net-(T1-C): track 35.4 -> 38.0 mm, vias 1 -> 2

Commit message: a
Parts:
- moved C5 0.59 mm to (136.0, 89.2)
Routing:
- net GND: track 96.4 -> 86.4 mm, vias 39 -> 46
Changed lines of the file:
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@@
 	(footprint "Capacitor_SMD:CP_Elec_6.3x7.7"
 		(layer "F.Cu")
-		(at 135.407121 89.21978)
+		(at 136 89.21978)
 		(descr "SMD capacitor, aluminum electrolytic, Nichicon, 6.3x7.7mm")
 		(tags "capacitor electrolytic")
@@
 		(tags "test point SMD pad")
 		(property "Reference" "TP24"
-			(at 0 1.648 0)
+			(at 3 0 0)
 			(layer "B.SilkS")
 			(effects
@@
 		(sheetname "/")
 		(sheetfile "Stylophon_1.kicad_sch")
-		(attr exclude_from_pos_files)
+		(attr exclude_from_pos_files exclude_from_bom)
 		(fp_circle
 			(center 0 0)
@@
 		(tags "test point SMD pad")
 		(property "Reference" "TP22"
-			(at 0 1.648 0)
+			(at 0 -2 0)
 			(layer "B.SilkS")
 			(effects
@@
 		(sheetname "/")
 		(sheetfile "Stylophon_1.kicad_sch")
-		(attr exclude_from_pos_files)
+		(attr exclude_from_pos_files exclude_from_bom)
 		(fp_circle
 			(center 0 0)
@@
 		(sheetname "/")
 		(sheetfile "Stylophon_1.kicad_sch")
-		(attr exclude_from_pos_files)
+		(attr exclude_from_pos_files exclude_from_bom)
 		(fp_circle
 			(center 0 0)
@@
 		(sheetname "/")
 		(sheetfile "Stylophon_1.kicad_sch")
-		(attr exclude_from_pos_files)
+		(attr exclude_from_pos_files exclude_from_bom)
 		(fp_circle
 			(center 0 0)
@@
 		(tags "test point SMD pad")
 		(property "Reference" "TP21"
-			(at 0 1.648 0)
+			(at -2.5 -0.6 0)
 			(layer "B.SilkS")
 			(effects
@@
 		(sheetname "/")
 		(sheetfile "Stylophon_1.kicad_sch")
-		(attr exclude_from_pos_files)
+		(attr exclude_from_pos_files exclude_from_bom)
 		(fp_circle
 			(center 0 0)
@@
 	)
 	(gr_text "mitg@htl-steyr.ac.at"
-		(at 92.9 105.2 90)
+		(at 169 83 0)
 		(layer "B.Cu" knockout)
 		(effects
@@
 	)
 	(segment
-		(start 137.16583 92.95395)
-		(end 140.9 89.21978)
-		(width 0.4)
-		(layer "F.Cu")
-		(net 17)
-	)
-	(segment
 		(start 148.875 92.405)
 		(end 148.875 94)
@@
 	)
 	(segment
-		(start 141.310749 92.95395)
-		(end 137.16583 92.95395)
-		(width 0.4)
-		(layer "F.Cu")
-		(net 17)
-	)
-	(segment
 		(start 123.32 86.92)
 		(end 123.4 87)
@@
 	)
 	(segment
-		(start 140.9 89.21978)
-		(end 140.9 86.55)
-		(width 0.4)
-		(layer "F.Cu")
-		(net 17)
-	)
-	(segment
 		(start 121.9 92.5)
 		(end 121.9 86.96)
@@
 	)
 	(segment
+		(start 140.9 89.21978)
+		(end 140.9 86.55)
+		(width 0.4)
+		(layer "F.Cu")
+		(net 17)
+	)
+	(segment
 		(start 131.35 79.5)
 		(end 131.35 77)
@@
 	)
 	(segment
-		(start 138.107121 89.21978)
+		(start 138.7 89.21978)
 		(end 140.9 89.21978)
 		(width 0.4)
@@
 	)
 	(via
-		(at 169 81)
+		(at 169 80)
 		(size 0.6)
 		(drill 0.4)
@@
 	)
 	(via
+		(at 132.9 77)
+		(size 0.6)
+		(drill 0.4)
+		(layers "F.Cu" "B.Cu")
+		(free yes)
+		(net 17)
+	)
+	(via
 		(at 159 76)
 		(size 0.6)
@@
 	)
 	(via
+		(at 169.482709 98.56329)
+		(size 0.6)
+		(drill 0.4)
+		(layers "F.Cu" "B.Cu")
+		(free yes)
+		(net 17)
+	)
+	(via
 		(at 165 76)
 		(size 0.6)
@@
 	)
 	(via
+		(at 115.270884 79.357523)
+		(size 0.6)
+		(drill 0.4)
+		(layers "F.Cu" "B.Cu")
+		(free yes)
+		(net 17)
+	)
+	(via
+		(at 117 81)
+		(size 0.6)
+		(drill 0.4)
+		(layers "F.Cu" "B.Cu")
+		(free yes)
+		(net 17)
+	)
+	(via
 		(at 154 95)
 		(size 0.6)
@@
 	)
 	(via
-		(at 169 84)
+		(at 169 85)
 		(size 0.6)
 		(drill 0.4)
@@
 	)
 	(via
-		(at 168 92)
+		(at 158.55 90.55)
+		(size 0.6)
+		(drill 0.4)
+		(layers "F.Cu" "B.Cu")
+		(free yes)
+		(net 17)
+	)
+	(via
+		(at 130 89)
 		(size 0.6)
 		(drill 0.4)
@@
 	)
 	(via
-		(at 132.409785 94.93682)
+		(at 115 99)
 		(size 0.6)
 		(drill 0.4)
@@
 	)
 	(via
-		(at 169 79)
+		(at 117 89)
 		(size 0.6)
 		(drill 0.4)
@@
 	)
 	(via
-		(at 162 76)
+		(at 169 89)
 		(size 0.6)
 		(drill 0.4)
@@
 	)
 	(via
+		(at 158 86)
+		(size 0.6)
+		(drill 0.4)
+		(layers "F.Cu" "B.Cu")
+		(free yes)
+		(net 17)
+	)
+	(via
+		(at 118.631632 99.002778)
+		(size 0.6)
+		(drill 0.4)
+		(layers "F.Cu" "B.Cu")
+		(free yes)
+		(net 17)
+	)
+	(via
 		(at 115 92)
 		(size 0.6)
@@
 	)
 	(via
-		(at 168 95)
+		(at 169 93)
 		(size 0.6)
 		(drill 0.4)

Commit message: title
Parts:
- moved TP3 0.10 mm to (163.0, 109.0)
Changed lines of the file:
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@@
 	)
 	(paper "A4")
+	(title_block
+		(title "Stylophone")
+		(rev "1.0")
+		(company "HTL Steyr")
+		(comment 1 "Gerrit Mitterhuemer")
+	)
 	(layers
 		(0 "F.Cu" signal)
@@
 	(footprint "Keypads:Keypad_Small"
 		(layer "F.Cu")
-		(at 163.1 109)
+		(at 163 109)
 		(descr "SMD rectangular pad as test Point, square 4.0mm side length")
 		(tags "test point SMD pad rectangle square")
