File: Stylophon_1.kicad_pcb (KiCad board)
At the start: 2 copper layers, 57 x 38.5 mm, 75 parts, among them J4 Stylus, SW1 On/Off, SW2 Vibrato, T1 BC846, T2 BC846, U1 NE555D

Commit message: Keyboard improvement
Parts:
- moved TP2 0.15 mm to (165.2, 104.4)
- moved TP4 0.10 mm to (160.4, 104.5)
Routing:
- net GND: track 86.4 -> 77.5 mm, vias 46 -> 59
Changed lines of the file:
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@@
 	(footprint "Keypads:Keypad_Small"
 		(layer "F.Cu")
-		(at 160.5 104.4)
+		(at 160.431908 104.468092)
 		(descr "SMD rectangular pad as test Point, square 4.0mm side length")
 		(tags "test point SMD pad rectangle square")
@@
 	(footprint "Keypads:Keypad_Small"
 		(layer "F.Cu")
-		(at 127.7 104.4)
+		(at 127.75 104.4)
 		(descr "SMD rectangular pad as test Point, square 4.0mm side length")
 		(tags "test point SMD pad rectangle square")
@@
 	(footprint "Keypads:Keypad_Small"
 		(layer "F.Cu")
-		(at 165.4 104.4)
+		(at 165.25 104.4)
 		(descr "SMD rectangular pad as test Point, square 4.0mm side length")
 		(tags "test point SMD pad rectangle square")
@@
 	)
 	(segment
+		(start 141.545649 93.18885)
+		(end 141.310749 92.95395)
+		(width 0.4)
+		(layer "F.Cu")
+		(net 17)
+	)
+	(segment
 		(start 166.9 90)
 		(end 163.9 90)
@@
 	)
 	(segment
-		(start 141.545649 95.278921)
-		(end 141.545649 93.18885)
-		(width 0.4)
-		(layer "F.Cu")
-		(net 17)
-	)
-	(segment
 		(start 157.85 92)
 		(end 154.1 92)
@@
 	)
 	(segment
-		(start 135 95.612821)
-		(end 135 95.513821)
-		(width 0.4)
-		(layer "F.Cu")
-		(net 17)
-	)
-	(segment
 		(start 123.4 87)
 		(end 123.36 86.96)
@@
 	)
 	(segment
-		(start 141.545649 93.18885)
-		(end 141.310749 92.95395)
-		(width 0.4)
-		(layer "F.Cu")
-		(net 17)
-	)
-	(segment
 		(start 122.82 86.92)
 		(end 122.78 86.96)
@@
 	)
 	(segment
-		(start 135 95.513821)
-		(end 141.310749 95.513821)
-		(width 0.4)
-		(layer "F.Cu")
-		(net 17)
-	)
-	(segment
 		(start 129.9 79.5)
 		(end 131.35 79.5)
@@
 	)
 	(segment
-		(start 141.310749 95.513821)
-		(end 141.545649 95.278921)
-		(width 0.4)
-		(layer "F.Cu")
-		(net 17)
-	)
-	(segment
 		(start 129.9 83.5)
 		(end 129.9 79.5)
@@
 	)
 	(via
+		(at 132.5 95.75)
+		(size 0.6)
+		(drill 0.4)
+		(layers "F.Cu" "B.Cu")
+		(free yes)
+		(net 17)
+	)
+	(via
 		(at 169 80)
 		(size 0.6)
@@
 	)
 	(via
+		(at 154.5 85)
+		(size 0.6)
+		(drill 0.4)
+		(layers "F.Cu" "B.Cu")
+		(free yes)
+		(net 17)
+	)
+	(via
 		(at 159 76)
 		(size 0.6)
@@
 	)
 	(via
+		(at 145.75 86.75)
+		(size 0.6)
+		(drill 0.4)
+		(layers "F.Cu" "B.Cu")
+		(free yes)
+		(net 17)
+	)
+	(via
 		(at 169.482709 98.56329)
 		(size 0.6)
@@
 	)
 	(via
+		(at 154.75 78.5)
+		(size 0.6)
+		(drill 0.4)
+		(layers "F.Cu" "B.Cu")
+		(free yes)
+		(net 17)
+	)
+	(via
 		(at 169 77)
 		(size 0.6)
@@
 	)
 	(via
+		(at 133.5 83.25)
+		(size 0.6)
+		(drill 0.4)
+		(layers "F.Cu" "B.Cu")
+		(free yes)
+		(net 17)
+	)
+	(via
 		(at 162 76)
 		(size 0.6)
@@
 	)
 	(via
+		(at 140.25 95.75)
+		(size 0.6)
+		(drill 0.4)
+		(layers "F.Cu" "B.Cu")
+		(free yes)
+		(net 17)
+	)
+	(via
 		(at 152 76)
 		(size 0.6)
@@
 	)
 	(via
+		(at 137.5 95.75)
+		(size 0.6)
+		(drill 0.4)
+		(layers "F.Cu" "B.Cu")
+		(free yes)
+		(net 17)
+	)
+	(via
 		(at 169 85)
 		(size 0.6)
@@
 	)
 	(via
+		(at 114.75 76.75)
+		(size 0.6)
+		(drill 0.4)
+		(layers "F.Cu" "B.Cu")
+		(free yes)
+		(net 17)
+	)
+	(via
 		(at 119 77)
 		(size 0.6)
@@
 	)
 	(via
-		(at 136 95.612821)
+		(at 130 95)
 		(size 0.6)
 		(drill 0.4)
@@
 	)
 	(via
-		(at 130 95)
+		(at 129 77)
 		(size 0.6)
 		(drill 0.4)
@@
 	)
 	(via
-		(at 129 77)
+		(at 136.5 78)
 		(size 0.6)
 		(drill 0.4)
@@
 	)
 	(via
+		(at 158.5 80)
+		(size 0.6)
+		(drill 0.4)
+		(layers "F.Cu" "B.Cu")
+		(free yes)
+		(net 17)
+	)
+	(via
 		(at 114.6 87.9)
 		(size 0.6)
@@
 	)
 	(via
+		(at 135 95.75)
+		(size 0.6)
+		(drill 0.4)
+		(layers "F.Cu" "B.Cu")
+		(free yes)
+		(net 17)
+	)
+	(via
 		(at 121 95)
 		(size 0.6)
@@
 	)
 	(via
+		(at 116 75.75)
+		(size 0.6)
+		(drill 0.4)
+		(layers "F.Cu" "B.Cu")
+		(free yes)
+		(net 17)
+	)
+	(via
 		(at 118.631632 99.002778)
 		(size 0.6)
@@
 	)
 	(via
+		(at 147.75 79)
+		(size 0.6)
+		(drill 0.4)
+		(layers "F.Cu" "B.Cu")
+		(free yes)
+		(net 17)
+	)
+	(via
 		(at 130 92)
 		(size 0.6)
@@
 	)
 	(via
+		(at 138.75 83.25)
+		(size 0.6)
+		(drill 0.4)
+		(layers "F.Cu" "B.Cu")
+		(free yes)
+		(net 17)
+	)
+	(via
 		(at 169 93)
 		(size 0.6)
@@
 	)
 	(segment
-		(start 162.999 102.099)
-		(end 164.534111 100.563889)
+		(start 161.9 109)
+		(end 162.849518 108.050482)
 		(width 0.4)
 		(layer "F.Cu")
@@
 	)
 	(segment
-		(start 161.9 109)
-		(end 162.999 107.901)
+		(start 162.849518 102.150482)
+		(end 164.436111 100.563889)
 		(width 0.4)
 		(layer "F.Cu")
@@
 	)
 	(segment
-		(start 162.999 107.901)
-		(end 162.999 102.099)
+		(start 164.436111 100.563889)
+		(end 165.069368 100.563889)
 		(width 0.4)
 		(layer "F.Cu")
@@
 	)
 	(segment
-		(start 164.534111 100.563889)
-		(end 165.069368 100.563889)
+		(start 162.849518 108.050482)
+		(end 162.849518 102.150482)
 		(width 0.4)
 		(layer "F.Cu")
@@
 	)
 	(segment
-		(start 162.337737 102.562263)
-		(end 162.337737 100.597222)
+		(start 160.5 104.4)
+		(end 160.5 102.434959)
 		(width 0.4)
 		(layer "F.Cu")
@@
 	)
 	(segment
-		(start 160.4 104.5)
-		(end 162.337737 102.562263)
+		(start 159.606105 97.647497)
+		(end 159.606105 97.488889)
 		(width 0.4)
 		(layer "F.Cu")
@@
 	)
 	(segment
-		(start 159.606105 97.647497)
-		(end 159.606105 97.488889)
+		(start 162.337737 100.379129)
+		(end 159.606105 97.647497)
 		(width 0.4)
 		(layer "F.Cu")
@@
 	)
 	(segment
-		(start 162.337737 100.379129)
-		(end 159.606105 97.647497)
+		(start 160.4 104.5)
+		(end 160.5 104.4)
+		(width 0.4)
+		(layer "F.Cu")
+		(net 21)
+	)
+	(segment
+		(start 160.5 102.434959)
+		(end 162.337737 100.597222)
 		(width 0.4)
 		(layer "F.Cu")

Commit message: Release V1.0
Parts:
- moved T1 0.51 mm to (131.8, 83.0)
- moved J4 0.25 mm to (156.9, 78.2)
Routing:
- net Net-(T1-C): track 38.0 -> 37.0 mm
- net Net-(T1-B): track 4.43 -> 4.98 mm
- net Net-(D1-A): track 6.33 -> 6.83 mm
- net GND: vias 59 -> 63
